File: PCB/reckoner.kicad_sch (KiCad schematic)
At the start: 0 parts

Commit message: Design the Reckoner: requirements, BOM and wired schematic
Parts:
- added C1, C2: 2.2uF 400V, Capacitor_SMD:CP_Elec_6.3x9.9, symbol Device:C_Polarized
- added C10, C12, C13, C14, C15, C16: 100nF, Capacitor_SMD:C_0402_1005Metric, symbol Device:C
- added C11, C8: 1uF, Capacitor_SMD:C_0402_1005Metric, symbol Device:C
- added C17, C18: 10nF, Capacitor_SMD:C_0402_1005Metric, symbol Device:C
- added C19: 100pF, Capacitor_SMD:C_0402_1005Metric, symbol Device:C
- added C3: 100nF X7R, Capacitor_SMD:C_0603_1608Metric, symbol Device:C
- added C4, C9: 22uF, Capacitor_SMD:C_0805_2012Metric, symbol Device:C
- added C5, C6: 22uF, Capacitor_SMD:C_1206_3216Metric, symbol Device:C
- added C7: 470uF 10V, Capacitor_SMD:CP_Elec_8x10, symbol Device:C_Polarized
- added D1: M7, Diode_SMD:D_SMA, symbol Device:D
- added D2, D3: ES1J, Diode_SMD:D_SMA, symbol Device:D
- added D4: red, LED_SMD:LED_0603_1608Metric, symbol Device:LED
- added D5, D6: 1N4148W, Diode_SMD:D_SOD-123, symbol Device:D
- added D7, D8, D9: BAT54S, Package_TO_SOT_SMD:SOT-23, symbol Diode:BAT54S
- added F1: 2A 250VAC 0443002.DR, Fuse:Fuse_Littelfuse-NANO2-462, symbol Device:Fuse
- added J1: L_IN, Connector_Wire:SolderWire-0.75sqmm_1x01_D1.25mm_OD2.3mm, symbol Connector_Generic:Conn_01x01
- added J2: N_IN, Connector_Wire:SolderWire-0.75sqmm_1x01_D1.25mm_OD2.3mm, symbol Connector_Generic:Conn_01x01
- added J3: S_UP, Connector_Wire:SolderWire-0.75sqmm_1x01_D1.25mm_OD2.3mm, symbol Connector_Generic:Conn_01x01
- added J4: S_DN, Connector_Wire:SolderWire-0.75sqmm_1x01_D1.25mm_OD2.3mm, symbol Connector_Generic:Conn_01x01
- added J5: M_UP, Connector_Wire:SolderWire-0.75sqmm_1x01_D1.25mm_OD2.3mm, symbol Connector_Generic:Conn_01x01
- added J6: M_DN, Connector_Wire:SolderWire-0.75sqmm_1x01_D1.25mm_OD2.3mm, symbol Connector_Generic:Conn_01x01
- added K1: HF46F-G/5-HS1, Relay_THT:Relay_SPST_Omron_G5NB, symbol Relay:Relay_SPST-NO
- added K2: G5Q-14 DC5, Relay_THT:Relay_SPDT_Omron-G5Q-1, symbol Relay:G5Q-1
- added L1: 1mH, Inductor_SMD:L_Taiyo-Yuden_NR-50xx, symbol Device:L
- added L2: 680uH, Inductor_THT:L_Radial_D8.7mm_P5.00mm_Fastron_07HCP, symbol Device:L
- added Q1, Q2: AO3400A, Package_TO_SOT_SMD:SOT-23, symbol Transistor_FET:Q_NMOS_GSD
- added R1: 10R 1W fusible, Resistor_THT:R_Axial_DIN0309_L9.0mm_D3.2mm_P2.54mm_Vertical, symbol Device:R
- added R10: 10mR 1W, Resistor_SMD:R_1206_3216Metric, symbol Device:R
- added R11, R12, R15: 1k, Resistor_SMD:R_0402_1005Metric, symbol Device:R
- added R13, R14, R22, R23: 1M 1206, Resistor_SMD:R_1206_3216Metric, symbol Device:R
- added R16, R17, R18, R19: 100k 1206, Resistor_SMD:R_1206_3216Metric, symbol Device:R
- added R2: 3.3k, Resistor_SMD:R_0402_1005Metric, symbol Device:R
- added R20, R21, R24: 1M, Resistor_SMD:R_0402_1005Metric, symbol Device:R
- added R25, R26, R27, R5, R6: 10k, Resistor_SMD:R_0402_1005Metric, symbol Device:R
- added R3: 2.2k, Resistor_SMD:R_0402_1005Metric, symbol Device:R
- added R4: 1.5k, Resistor_SMD:R_0603_1608Metric, symbol Device:R
- added R7: 1k, Resistor_SMD:R_0603_1608Metric, symbol Device:R
- added R8, R9: 100k, Resistor_SMD:R_0402_1005Metric, symbol Device:R
- added RV1: S07K275, Varistor:RV_Disc_D7mm_W5.5mm_P5mm, symbol Device:Varistor
- added TP1: +5V/VBUS, TestPoint:TestPoint_Pad_D1.0mm, symbol Connector:TestPoint
- added TP10: IO0, TestPoint:TestPoint_Pad_D1.0mm, symbol Connector:TestPoint
- added TP11: IO1, TestPoint:TestPoint_Pad_D1.0mm, symbol Connector:TestPoint
- added TP12: IO14, TestPoint:TestPoint_Pad_D1.0mm, symbol Connector:TestPoint
- added TP13: IO22, TestPoint:TestPoint_Pad_D1.0mm, symbol Connector:TestPoint
- added TP2: GND, TestPoint:TestPoint_Pad_D1.0mm, symbol Connector:TestPoint
- added TP3: USB_DP, TestPoint:TestPoint_Pad_D1.0mm, symbol Connector:TestPoint
- added TP4: USB_DM, TestPoint:TestPoint_Pad_D1.0mm, symbol Connector:TestPoint
- added TP5: BOOT, TestPoint:TestPoint_Pad_D1.0mm, symbol Connector:TestPoint
- added TP6: EN, TestPoint:TestPoint_Pad_D1.0mm, symbol Connector:TestPoint
- added TP7: TXD0, TestPoint:TestPoint_Pad_D1.0mm, symbol Connector:TestPoint
- added TP8: RXD0, TestPoint:TestPoint_Pad_D1.0mm, symbol Connector:TestPoint
- added TP9: +3V3, TestPoint:TestPoint_Pad_D1.0mm, symbol Connector:TestPoint
- added U1: LNK3206D, Package_SO:PowerIntegrations_SO-8C, symbol Regulator_Switching:LNK3202D
- added U2: AP2112K-3.3, Package_TO_SOT_SMD:SOT-23-5, symbol Regulator_Linear:TPS76316
- added U3: ESP32-C6-MINI-1-N4, RF_Module:ESP32-C6-MINI-1, symbol RF_Module:ESP32-C6-MINI-1
- added U4: HLW8110, Package_SO:SOIC-8_3.9x4.9mm_P1.27mm, symbol reckoner:HLW8110
Connections:
- new net +3V3: C10.1, C16.1, C9.1, D7.2 (K), D8.2 (K), D9.2 (K), R20.1, R21.1, R5.1, R6.1, TP9.1, U2.5 (VOUT), U3.3 (3V3), U4.8 (VDD)
- new net +5V: C5.1, C6.1, C7.1, C8.1, D3.2 (A), D5.1 (K), D6.1 (K), K1.A1, K2.1, L2.2, R4.1, TP1.1, U2.1 (VIN), U2.3 (EN)
- new net BOOT: TP5.1, U3.23 (IO9)
- new net BP: C3.1, U1.1 (BP/M)
- new net EN: C11.1, R5.2, TP6.1, U3.8 (EN)
- new net FB: R2.2, R3.1, U1.2 (FB)
- new net FB_HOLD: C4.1, D3.1 (K), R2.1
- new net GND: C1.2, C10.2, C11.2, C12.2, C13.2, C14.2, C15.2, C16.2, C17.2, C18.2, C19.2, C2.2, C5.2, C6.2, C7.2, C8.2, C9.2, D2.2 (A), D4.1 (K), D7.1 (A), D8.1 (A), D9.1 (A), F1.2, Q1.2 (S), Q2.2 (S), R10.1, R12.1, R15.2, R24.2, R4.2, R8.2, R9.2, RV1.2, TP2.1, U2.2 (GND), U3.1 (GND), U3.11 (GND), U3.14 (GND), U3.2 (GND), U3.36 (GND), U3.37 (GND), U3.38 (GND), U3.39 (GND), U3.40 (GND), U3.41 (GND), U3.42 (GND), U3.43 (GND), U3.44 (GND), U3.45 (GND), U3.46 (GND), U3.47 (GND), U3.48 (GND), U3.49 (GND), U3.50 (GND), U3.51 (GND), U3.52 (GND), U3.53 (GND), U4.4 (GND)
- new net HV_BUS: C2.1, L1.2, U1.4 (D)
- new net HV_RAW: C1.1, D1.1 (K), L1.1
- new net IAN: C13.1, R12.2, U4.2 (IAN)
- new net IAP: C12.1, R11.2, U4.1 (IAP)
- new net IO0: TP10.1, U3.12 (IO0)
- new net IO1: TP11.1, U3.13 (IO1)
- new net IO14: TP12.1, U3.19 (IO14)
- new net IO22: TP13.1, U3.28 (IO22)
- new net IO8: R6.2, U3.22 (IO8)
- new net K1_COIL: D5.2 (A), K1.A2, Q1.3 (D)
- new net K1_DRV: Q1.1 (G), R8.1, U3.24 (IO18)
- new net K2_COIL: D6.2 (A), K2.5, Q2.3 (D)
- new net K2_DRV: Q2.1 (G), R9.1, U3.25 (IO19)
- new net LED_A: D4.2 (A), R7.2
- new net LED_IO: R7.1, U3.29 (IO23)
- new net L_IN: F1.1, J1.1 (Pin_1)
- new net L_K1: K1.14, K2.2
- new net L_SH: K1.13, R10.2, R11.1
- new net MTR_RX: U3.26 (IO20), U4.6 (TX)
- new net MTR_TX: U3.27 (IO21), U4.7 (RX)
- new net M_DN: J6.1 (Pin_1), K2.4
- new net M_UP: J5.1 (Pin_1), K2.3
- new net N_IN: J2.1 (Pin_1), R1.1, R13.1, R22.1, RV1.1
- new net N_RF: D1.2 (A), R1.2
- new net RXD0: TP8.1, U3.30 (RXD0)
- new net SDN: C18.1, D8.3 (COM), R19.2, R21.2, R26.1
- new net SDN_IO: R26.2, U3.6 (IO3)
- new net SUP: C17.1, D7.3 (COM), R17.2, R20.2, R25.1
- new net SUP_IO: R25.2, U3.5 (IO2)
- new net SW: C3.2, C4.2, D2.1 (K), L2.1, R3.2, U1.5 (S), U1.6 (S), U1.7 (S), U1.8 (S)
- new net S_DN: J4.1 (Pin_1), R18.1
- new net S_DN_MID: R18.2, R19.1
- new net S_UP: J3.1 (Pin_1), R16.1
- new net S_UP_MID: R16.2, R17.1
- new net TXD0: TP7.1, U3.31 (TXD0)
- new net USB_DM: TP4.1, U3.17 (IO12)
- new net USB_DP: TP3.1, U3.18 (IO13)
- new net VP: C14.1, R14.2, R15.1, U4.3 (VP)
- new net VP_MID: R13.2, R14.1
- new net VREF: C15.1, U4.5 (VREF)
- new net ZX: C19.1, D9.3 (COM), R23.2, R24.1, R27.1
- new net ZX_IO: R27.2, U3.16 (IO7)
- new net ZX_MID: R22.2, R23.1
- no-connect marks 0 -> 12
Other:
- note added: "3.3 V regulator"
- note added: "Button inputs and mains zero-cross sense"
- note added: "Flash only with mains disconnected (USB on TP1, TP2, TP3, TP4)."
- note added: "GND = mains L after F1. Non-isolated: every node is LIVE when powered."
- note added: "K1 makes and breaks the load; K2 (NO = UP, NC = DOWN) changes only while K1 is open."
- note added: "Mains input"
- note added: "Microcontroller"
- note added: "Motor current and mains voltage metering"
- note added: "Motor relays"
- note added: "Off-line 5 V supply"
- note added: "Programming and test pads"

Commit message: Change C2 to FOLLON 3.9 µF 400 V for ripple current
The LNK3206's drain pulses put about 45 mA RMS into C2, 239 % of the
Honor 2.2 µF part's rating. The FOLLON EFVD400ADA3R9M08B0 (C33129636,
8 x 10.5 mm, CP_Elec_8x10) runs at about 49 %. C1 is unchanged.
Hold-up in the README corrected to the worst-case figure.
Parts:
- C2: value 2.2uF 400V -> 3.9uF 400V; footprint Capacitor_SMD:CP_Elec_6.3x9.9 -> Capacitor_SMD:CP_Elec_8x10; LCSC C48970947 -> C33129636
Changed lines of the file:
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@@
 			)
 		)
-		(property "Value" "2.2uF 400V"
+		(property "Value" "3.9uF 400V"
 			(at 135.89 68.9609 0)
 			(show_name no)
@@
 			)
 		)
-		(property "Footprint" "Capacitor_SMD:CP_Elec_6.3x9.9"
+		(property "Footprint" "Capacitor_SMD:CP_Elec_8x10"
 			(at 144.78 71.12 0)
 			(hide yes)
@@
 			)
 		)
-		(property "LCSC" "C48970947"
+		(property "LCSC" "C33129636"
 			(at 144.78 71.12 0)
 			(hide yes)
@@
 		)
 	)
+	(symbol_instances
+		(path "/a4d88e87-23e2-4ab8-853d-15d5cb8e46f0/9b38a59f-1916-4da2-bbd8-d49cd447b223"
+			(reference "C2")
+			(unit 1)
+			(value "3.9uF 400V")
+			(footprint "Capacitor_SMD:CP_Elec_8x10")
+		)
+)
 	(sheet_instances
 		(path "/"

Commit message: Use LCSC footprints for F1, RV1 and L2
Parts:
- F1: footprint Fuse:Fuse_Littelfuse-NANO2-462 -> EasyEDA:FUSE-SMD_L10.1-W3.1
- L2: footprint Inductor_THT:L_Radial_D8.7mm_P5.00mm_Fastron_07HCP -> EasyEDA:IND-TH_BD9.5-P5.20-D0.6
- RV1: footprint Varistor:RV_Disc_D7mm_W5.5mm_P5mm -> EasyEDA:RES-TH_L9.0-W4.6-P5.00-D0.6-S1.60
Changed lines of the file:
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@@
 			)
 		)
-		(property "Footprint" "Inductor_THT:L_Radial_D8.7mm_P5.00mm_Fastron_07HCP"
+		(property "Footprint" "EasyEDA:IND-TH_BD9.5-P5.20-D0.6"
 			(at 215.9 58.42 0)
 			(hide yes)
@@
 			)
 		)
-		(property "Footprint" "Varistor:RV_Disc_D7mm_W5.5mm_P5mm"
+		(property "Footprint" "EasyEDA:RES-TH_L9.0-W4.6-P5.00-D0.6-S1.60"
 			(at 64.77 60.96 0)
 			(hide yes)
@@
 			)
 		)
-		(property "Footprint" "Fuse:Fuse_Littelfuse-NANO2-462"
+		(property "Footprint" "EasyEDA:FUSE-SMD_L10.1-W3.1"
 			(at 40.64 50.8 0)
 			(hide yes)
@@
 			(footprint "Capacitor_SMD:CP_Elec_8x10")
 		)
+		(path "/a4d88e87-23e2-4ab8-853d-15d5cb8e46f0/ff7819d0-4648-4566-9bc7-334491019cea"
+			(reference "F1")
+			(unit 1)
+			(value "2A 250VAC 0443002.DR")
+			(footprint "EasyEDA:FUSE-SMD_L10.1-W3.1")
+		)
+		(path "/a4d88e87-23e2-4ab8-853d-15d5cb8e46f0/152ad465-2165-4621-9081-1c0d35cffb24"
+			(reference "RV1")
+			(unit 1)
+			(value "S07K275")
+			(footprint "EasyEDA:RES-TH_L9.0-W4.6-P5.00-D0.6-S1.60")
+		)
+		(path "/a4d88e87-23e2-4ab8-853d-15d5cb8e46f0/0ee01271-869c-4a67-a81b-cb33e7fd130f"
+			(reference "L2")
+			(unit 1)
+			(value "680uH")
+			(footprint "EasyEDA:IND-TH_BD9.5-P5.20-D0.6")
+		)
 )

Commit message: Place and route the board
Other:
- company: (none) -> KOZELJ Michele
- title: (none) -> Reckoner
Changed lines of the file:
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@@
 	(generator_version "10.0")
 	(paper "A3")
+	(title_block
+		(title "Reckoner")
+		(company "KOZELJ Michele")
+	)
 	(text "Microcontroller"
 		(exclude_from_sim no)
@@
 		)
 	)
-	(symbol_instances
-		(path "/a4d88e87-23e2-4ab8-853d-15d5cb8e46f0/9b38a59f-1916-4da2-bbd8-d49cd447b223"
-			(reference "C2")
-			(unit 1)
-			(value "3.9uF 400V")
-			(footprint "Capacitor_SMD:CP_Elec_8x10")
-		)
-		(path "/a4d88e87-23e2-4ab8-853d-15d5cb8e46f0/ff7819d0-4648-4566-9bc7-334491019cea"
-			(reference "F1")
-			(unit 1)
-			(value "2A 250VAC 0443002.DR")
-			(footprint "EasyEDA:FUSE-SMD_L10.1-W3.1")
-		)
-		(path "/a4d88e87-23e2-4ab8-853d-15d5cb8e46f0/152ad465-2165-4621-9081-1c0d35cffb24"
-			(reference "RV1")
-			(unit 1)
-			(value "S07K275")
-			(footprint "EasyEDA:RES-TH_L9.0-W4.6-P5.00-D0.6-S1.60")
-		)
-		(path "/a4d88e87-23e2-4ab8-853d-15d5cb8e46f0/0ee01271-869c-4a67-a81b-cb33e7fd130f"
-			(reference "L2")
-			(unit 1)
-			(value "680uH")
-			(footprint "EasyEDA:IND-TH_BD9.5-P5.20-D0.6")
-		)
-)
 	(sheet_instances
 		(path "/"
