File: PCB/reckoner.kicad_pcb (KiCad board)
At the start: 2 copper layers, 0 parts

Commit message: Place and route the board
Parts:
- added C1: 2.2uF 400V, Capacitor_SMD:CP_Elec_6.3x9.9, F.Cu at (102.5, 105.5)
- added C10: 100nF, Capacitor_SMD:C_0402_1005Metric, F.Cu at (146.4, 114.4)
- added C11: 1uF, Capacitor_SMD:C_0402_1005Metric, F.Cu at (141.4, 114.2)
- added C12: 100nF, Capacitor_SMD:C_0402_1005Metric, F.Cu at (97.5, 118.5)
- added C13: 100nF, Capacitor_SMD:C_0402_1005Metric, F.Cu at (95.0, 122.0)
- added C14: 100nF, Capacitor_SMD:C_0402_1005Metric, F.Cu at (95.5, 125.0)
- added C15: 100nF, Capacitor_SMD:C_0402_1005Metric, F.Cu at (99.0, 127.0)
- added C16: 100nF, Capacitor_SMD:C_0402_1005Metric, F.Cu at (105.0, 121.5)
- added C17: 10nF, Capacitor_SMD:C_0402_1005Metric, F.Cu at (128.0, 137.5)
- added C18: 10nF, Capacitor_SMD:C_0402_1005Metric, F.Cu at (136.5, 136.0)
- added C19: 100pF, Capacitor_SMD:C_0402_1005Metric, F.Cu at (92.5, 135.0)
- added C2: 3.9uF 400V, Capacitor_SMD:CP_Elec_8x10, F.Cu at (121.5, 106.5)
- added C3: 100nF X7R, Capacitor_SMD:C_0603_1608Metric, F.Cu at (132.5, 106.5)
- added C4: 22uF, Capacitor_SMD:C_0805_2012Metric, F.Cu at (137.0, 102.0)
- added C5: 22uF, Capacitor_SMD:C_1206_3216Metric, F.Cu at (122.5, 118.5)
- added C6: 22uF, Capacitor_SMD:C_1206_3216Metric, F.Cu at (122.5, 123.5)
- added C7: 470uF 10V, Capacitor_SMD:CP_Elec_8x10, F.Cu at (111.0, 118.0)
- added C8: 1uF, Capacitor_SMD:C_0402_1005Metric, F.Cu at (141.0, 110.0)
- added C9: 22uF, Capacitor_SMD:C_0805_2012Metric, F.Cu at (148.4, 112.9)
- added D1: M7, Diode_SMD:D_SMA, F.Cu at (95.0, 106.5)
- added D2: ES1J, Diode_SMD:D_SMA, F.Cu at (133.0, 112.0)
- added D3: ES1J, Diode_SMD:D_SMA, F.Cu at (142.5, 104.0)
- added D4: red, LED_SMD:LED_0603_1608Metric, F.Cu at (147.5, 131.2)
- added D5: 1N4148W, Diode_SMD:D_SOD-123, F.Cu at (123.5, 135.0)
- added D6: 1N4148W, Diode_SMD:D_SOD-123, F.Cu at (123.5, 144.0)
- added D7: BAT54S, Package_TO_SOT_SMD:SOT-23, F.Cu at (132.6, 134.1)
- added D8: BAT54S, Package_TO_SOT_SMD:SOT-23, F.Cu at (139.0, 134.1)
- added D9: BAT54S, Package_TO_SOT_SMD:SOT-23, F.Cu at (89.0, 135.0)
- added F1: 2A 250VAC 0443002.DR, EasyEDA:FUSE-SMD_L10.1-W3.1, F.Cu at (91.5, 114.5)
- added J1: L_IN, Connector_Wire:SolderWire-0.75sqmm_1x01_D1.25mm_OD2.3mm, F.Cu at (84.0, 118.5)
- added J2: N_IN, Connector_Wire:SolderWire-0.75sqmm_1x01_D1.25mm_OD2.3mm, F.Cu at (84.0, 105.0)
- added J3: S_UP, Connector_Wire:SolderWire-0.75sqmm_1x01_D1.25mm_OD2.3mm, F.Cu at (132.5, 149.0)
- added J4: S_DN, Connector_Wire:SolderWire-0.75sqmm_1x01_D1.25mm_OD2.3mm, F.Cu at (139.0, 149.0)
- added J5: M_UP, Connector_Wire:SolderWire-0.75sqmm_1x01_D1.25mm_OD2.3mm, F.Cu at (85.0, 148.5)
- added J6: M_DN, Connector_Wire:SolderWire-0.75sqmm_1x01_D1.25mm_OD2.3mm, F.Cu at (93.0, 148.5)
- added K1: HF46F-G/5-HS1, Relay_THT:Relay_SPST_Omron_G5NB, F.Cu at (120.0, 135.8)
- added K2: G5Q-14 DC5, Relay_THT:Relay_SPDT_Omron-G5Q-1, F.Cu at (119.4, 141.2)
- added L1: 1mH, Inductor_SMD:L_Taiyo-Yuden_NR-50xx, F.Cu at (109.8, 105.5)
- added L2: 680uH, EasyEDA:IND-TH_BD9.5-P5.20-D0.6, F.Cu at (129.5, 119.1)
- added Q1: AO3400A, Package_TO_SOT_SMD:SOT-23, F.Cu at (123.4, 129.0)
- added Q2: AO3400A, Package_TO_SOT_SMD:SOT-23, F.Cu at (124.1, 150.6)
- added R1: 10R 1W fusible, Resistor_THT:R_Axial_DIN0309_L9.0mm_D3.2mm_P2.54mm_Vertical, F.Cu at (88.1, 102.5)
- added R10: 10mR 1W, Resistor_SMD:R_1206_3216Metric, F.Cu at (103.0, 118.5)
- added R11: 1k, Resistor_SMD:R_0402_1005Metric, F.Cu at (99.5, 118.5)
- added R12: 1k, Resistor_SMD:R_0402_1005Metric, F.Cu at (93.5, 122.0)
- added R13: 1M 1206, Resistor_SMD:R_1206_3216Metric, F.Cu at (86.0, 125.0)
- added R14: 1M 1206, Resistor_SMD:R_1206_3216Metric, F.Cu at (91.0, 125.0)
- added R15: 1k, Resistor_SMD:R_0402_1005Metric, F.Cu at (94.0, 125.0)
- added R16: 100k 1206, Resistor_SMD:R_1206_3216Metric, F.Cu at (132.5, 143.5)
- added R17: 100k 1206, Resistor_SMD:R_1206_3216Metric, F.Cu at (132.5, 138.5)
- added R18: 100k 1206, Resistor_SMD:R_1206_3216Metric, F.Cu at (139.0, 143.5)
- added R19: 100k 1206, Resistor_SMD:R_1206_3216Metric, F.Cu at (139.0, 138.5)
- added R2: 3.3k, Resistor_SMD:R_0402_1005Metric, F.Cu at (133.0, 100.5)
- added R20: 1M, Resistor_SMD:R_0402_1005Metric, F.Cu at (128.0, 136.5)
- added R21: 1M, Resistor_SMD:R_0402_1005Metric, F.Cu at (143.0, 137.0)
- added R22: 1M 1206, Resistor_SMD:R_1206_3216Metric, F.Cu at (83.0, 128.5)
- added R23: 1M 1206, Resistor_SMD:R_1206_3216Metric, F.Cu at (88.0, 130.0)
- added R24: 1M, Resistor_SMD:R_0402_1005Metric, F.Cu at (92.5, 134.0)
- added R25: 10k, Resistor_SMD:R_0402_1005Metric, F.Cu at (133.5, 131.5)
- added R26: 10k, Resistor_SMD:R_0402_1005Metric, F.Cu at (142.0, 132.5)
- added R27: 10k, Resistor_SMD:R_0402_1005Metric, F.Cu at (94.5, 130.0)
- added R3: 2.2k, Resistor_SMD:R_0402_1005Metric, F.Cu at (131.0, 102.0)
- added R4: 1.5k, Resistor_SMD:R_0603_1608Metric, F.Cu at (116.2, 124.0)
- added R5: 10k, Resistor_SMD:R_0402_1005Metric, F.Cu at (142.9, 114.2)
- added R6: 10k, Resistor_SMD:R_0402_1005Metric, F.Cu at (135.5, 125.5)
- added R7: 1k, Resistor_SMD:R_0603_1608Metric, F.Cu at (145.5, 131.2)
- added R8: 100k, Resistor_SMD:R_0402_1005Metric, F.Cu at (125.0, 131.5)
- added R9: 100k, Resistor_SMD:R_0402_1005Metric, F.Cu at (127.5, 151.5)
- added RV1: S07K275, EasyEDA:RES-TH_L9.0-W4.6-P5.00-D0.6-S1.60, F.Cu at (86.5, 109.5)
- added TP1: +5V/VBUS, TestPoint:TestPoint_Pad_D1.0mm, F.Cu at (147.5, 100.5)
- added TP10: IO0, TestPoint:TestPoint_Pad_D1.0mm, B.Cu at (137.0, 115.5)
- added TP11: IO1, TestPoint:TestPoint_Pad_D1.0mm, B.Cu at (136.0, 119.5)
- added TP12: IO14, TestPoint:TestPoint_Pad_D1.0mm, F.Cu at (146.5, 149.6)
- added TP13: IO22, TestPoint:TestPoint_Pad_D1.0mm, F.Cu at (146.5, 145.0)
- added TP2: GND, TestPoint:TestPoint_Pad_D1.0mm, F.Cu at (148.0, 107.5)
- added TP3: USB_DP, TestPoint:TestPoint_Pad_D1.0mm, B.Cu at (136.0, 125.0)
- added TP4: USB_DM, TestPoint:TestPoint_Pad_D1.0mm, B.Cu at (136.0, 129.5)
- added TP5: BOOT, TestPoint:TestPoint_Pad_D1.0mm, F.Cu at (139.5, 107.5)
- added TP6: EN, TestPoint:TestPoint_Pad_D1.0mm, B.Cu at (140.0, 112.5)
- added TP7: TXD0, TestPoint:TestPoint_Pad_D1.0mm, B.Cu at (147.0, 140.0)
- added TP8: RXD0, TestPoint:TestPoint_Pad_D1.0mm, B.Cu at (147.0, 135.4)
- added TP9: +3V3, TestPoint:TestPoint_Pad_D1.0mm, B.Cu at (148.0, 105.5)
- added U1: LNK3206D, Package_SO:PowerIntegrations_SO-8C, F.Cu at (128.9, 106.3)
- added U2: AP2112K-3.3, Package_TO_SOT_SMD:SOT-23-5, F.Cu at (144.0, 109.9)
- added U3: ESP32-C6-MINI-1-N4, RF_Module:ESP32-C6-MINI-1, F.Cu at (144.0, 122.4)
- added U4: HLW8110, Package_SO:SOIC-8_3.9x4.9mm_P1.27mm, F.Cu at (100.0, 123.4)
Routing:
- net GND: track 0.00 -> 391.7 mm, vias 0 -> 23
- net +3V3: track 0.00 -> 152.0 mm, vias 0 -> 12
- net +5V: track 0.00 -> 96.5 mm, vias 0 -> 4
- net /MTR_TX: track 0.00 -> 49.9 mm
- net /K2_DRV: track 0.00 -> 48.8 mm, vias 0 -> 2
- net /ZX_IO: track 0.00 -> 47.9 mm, vias 0 -> 2
- net /MTR_RX: track 0.00 -> 44.0 mm
- net /SW: track 0.00 -> 40.0 mm
- net /N_IN: track 0.00 -> 36.3 mm, vias 0 -> 1
- net /IO14: track 0.00 -> 31.0 mm, vias 0 -> 2
- net /SUP_IO: track 0.00 -> 28.1 mm, vias 0 -> 2
- net /L_SH: track 0.00 -> 23.2 mm, vias 0 -> 3
- net /BOOT: track 0.00 -> 22.2 mm, vias 0 -> 2
- net /M_UP: track 0.00 -> 21.1 mm
- net /SDN_IO: track 0.00 -> 19.6 mm, vias 0 -> 2
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- added copper zone on B.Cu, net GND
- added copper zone on F.Cu, net GND
Other:
- board outline added: 70 x 54.5 mm

Commit message: Add silkscreen artwork: mains warnings, licence and QR code
Parts:
- added G***: LOGO, LOGO, F.Cu at (83.5, 139.0)
- added G***: LOGO, LOGO, B.Cu at (117.5, 106.5)
- added G***: LOGO, LOGO, B.Cu at (99.0, 114.5)
- added G***: LOGO, LOGO, B.Cu at (118.0, 122.5)
- added G***: LOGO, LOGO, B.Cu at (90.0, 136.0)
- added G***: LOGO, LOGO, B.Cu at (134.5, 139.5)
Other:
- board text added: "JLCJLCJLCJLC"
